File: Z31HELLEN.kicad_pcb (KiCad board)
At the start: 2 copper layers, 180.2 x 188.2 mm, 2 parts, among them J6 172023-1

Commit message: Add files via upload
Parts:
- removed J5: ~, Yon:Connector 1
- removed J6: 172023-1, Yon:1720231
- added CON1: , Z31:Z31 15 + 36, F.Cu at (181.2, 223.5)
- added Z31: ~, Z31:Z31 15 + 36, F.Cu at (81.2, 15.0)

Commit message: Add files via upload
Parts:
- removed CON1: , Z31:Z31 15 + 36
- moved Z31 231.2 mm to (181.1, 223.5)
Other:
- outline, holes or cut-outs redrawn
